File: hardware/bis-bajak-laut.kicad_pcb (KiCad board)
At the start: 2 copper layers, 253 parts, among them J1 TFT, J2 USB_C_Receptacle_USB2.0_14P, J3 ProgHeader, J4 BIS BAJAK LAUT IO, J5 BIS BAJAK LAUT IO, Q1 SI2301, Q10 SI2301, Q11 MMBT3906, Q12 BCM857, Q13 MMBT3906, Q14 SI2301, Q2 SI2301, Q3 SI2301, Q4 SI2301, Q5 SI2301, Q6 SI2301, Q7 SI2301, Q8 MMBT7002K, Q9 SI2301, SW1 W25Sel, SW2 BUTTON, U1 MT29F1G01ABAFDWB, U10 LMV331, U11 AP2127K-ADJ, U12 LMV321, U13 LMV321, U14 W25Q128JVS, U15 AMS1117-3.3, U16 SN74LVC1T45DRL, U17 SN74LVC1T45DRL, U18 SN74LVC1T45DRL, U19 SN74LVC1T45DRL, U2 74HC595, U20 SN74LVC1T45DRL, U21 SN74LVC1T45DRL, U22 SN74LVC1T45DRL, U23 SN74LVC1T45DRL, U3 LMV324, U4 CD74HC4067M, U5 74HC245, U6 74HC595, U7 LMV324, U8 LMV324, U9 RP2040, Y1 12Mhz

Commit message: feat: component arrangement progress 1
Parts:
- J3: moved to B.Cu
- moved R2 184.8 mm to (135.9, 408.9)
- moved R3 183.9 mm to (135.9, 410.9)
- moved R4 183.1 mm to (135.9, 412.9)
- moved R5 182.2 mm to (135.9, 414.9)
- moved R6 181.4 mm to (135.9, 416.9)
- moved U20 180.7 mm to (497.5, 36.2)
- moved R1 177.1 mm to (102.3, 409.8), turned to -90 degrees
- moved C48 176.4 mm to (497.7, 31.8)
- moved C47 173.6 mm to (497.7, 33.8)
- moved U8 168.7 mm to (142.5, 389.0)
- moved U16 166.3 mm to (462.4, 23.8)
- moved J1 164.0 mm to (117.4, 398.4), turned to -90 degrees
- moved U3 162.1 mm to (86.7, 389.9)
- moved R39 160.8 mm to (137.3, 390.8), turned to -90 degrees
- moved R25 160.3 mm to (117.6, 390.4), turned to 180 degrees
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