File: hardware/bis-bajak-laut.kicad_sch (KiCad schematic)
At the start: 253 parts, among them J1 TFT, J2 USB_C_Receptacle_USB2.0_14P, J3 ProgHeader, J4 BIS BAJAK LAUT IO, J5 BIS BAJAK LAUT IO, Q1 Q_PMOS_GSD, Q10 SI2301, Q11 MMBT3906, Q12 BCM857, Q13 MMBT3906, Q14 SI2301, Q2 Q_PMOS_GSD, Q3 Q_PMOS_GSD, Q4 Q_PMOS_GSD, Q5 Q_PMOS_GSD, Q6 Q_PMOS_GSD, Q7 Q_PMOS_GSD, Q8 Q_NMOS_GSD, Q9 Q_PMOS_GSD, SW1 W25Sel, SW2 BUTTON, U1 MT29F1G01ABAFDWB, U10 LMV331, U11 AP2127K-ADJ, U12 LMV321, U13 LMV321, U14 W25Q128JVS, U15 AMS1117-3.3, U16 SN74LVC1T45DRL, U17 SN74LVC1T45DRL, U18 SN74LVC1T45DRL, U19 SN74LVC1T45DRL, U2 74HC595, U20 SN74LVC1T45DRL, U21 SN74LVC1T45DRL, U22 SN74LVC1T45DRL, U23 SN74LVC1T45DRL, U3 LMV324, U4 CD74HC4067M, U5 74HC245, U6 74HC595, U7 LMV324, U8 LMV324, U9 RP2040, Y1 12Mhz

Commit message: feat: match footprint
Parts:
- C1, C10, C11, C12, C13, C14, C15, C16, C17, C18, C19, C2, C20, C21, C22, C23, C24, C25, C26, C27, C28, C29, C3, C30, C31, C32, C33, C34, C35, C36, C37, C38, C39, C4, C40, C41, C42, C43, C44, C45, C46, C47, C48, C49, C5, C50, C51, C52, C53, C54, C55, C56, C57, C58, C59, C6, C60, C61, C62, C63, C64, C65, C66, C67, C68, C69, C7, C70, C71, C72, C8, C9: footprint Capacitor_SMD:C_0805_2012Metric_Pad1.18x1.45mm_HandSolder -> Capacitor_SMD:C_0805_2012Metric
- D10: footprint LED_SMD:LED_1206_3216Metric_Pad1.42x1.75mm_HandSolder -> LED_SMD:LED_1206_3216Metric
- D2, D3, D4, D5, D6: footprint (none) -> Package_TO_SOT_SMD:SOT-523
- D7, D8, D9: footprint Diode_SMD:D_SOD-123 -> Diode_SMD:D_SOD-323
- J1: footprint (none) -> Connector_PinSocket_2.54mm:PinSocket_1x09_P2.54mm_Vertical
- J2: footprint (none) -> Connector_USB:USB_C_Receptacle_GCT_USB4110
- J3: footprint (none) -> Connector_PinSocket_2.54mm:PinSocket_1x03_P2.54mm_Vertical
- Q1, Q2, Q3, Q4, Q5, Q6, Q7, Q9: value Q_PMOS_GSD -> SI2301; footprint (none) -> Package_TO_SOT_SMD:SOT-23
- Q10, Q14: footprint (none) -> Package_TO_SOT_SMD:SOT-23
- Q8: value Q_NMOS_GSD -> MMBT7002K; footprint (none) -> Package_TO_SOT_SMD:SOT-23
- R1, R10, R100, R101, R102, R103, R104, R105, R106, R107, R108, R11, R12, R13, R14, R15, R16, R17, R18, R19, R2, R20, R21, R22, R23, R24, R25, R26, R27, R28, R29, R3, R30, R31, R32, R33, R34, R35, R36, R37, R38, R39, R4, R40, R41, R42, R43, R44, R45, R46, R47, R48, R49, R5, R50, R51, R52, R53, R54, R55, R56, R57, R58, R59, R6, R60, R61, R62, R63, R64, R65, R66, R67, R68, R69, R7, R70, R71, R72, R73, R74, R75, R76, R77, R78, R79, R8, R80, R81, R82, R83, R84, R85, R86, R87, R88, R89, R9, R90, R91, R92, R93, R94, R95, R96, R97, R98, R99: footprint Resistor_SMD:R_0805_2012Metric_Pad1.20x1.40mm_HandSolder -> Resistor_SMD:R_0805_2012Metric
- SW1, SW2: footprint (none) -> Button_Switch_SMD:SW_Push_1P1T_NO_6x6mm_H9.5mm
- U1: footprint dp-memory:U-PDFN-8 -> Package_DFN_QFN:W-PDFN-8-1EP_6x5mm_P1.27mm_EP3x3mm
- U10: footprint Package_TO_SOT_SMD:SOT-23-5_HandSoldering -> Package_TO_SOT_SMD:SOT-23-5
- U12, U13: footprint (none) -> Package_TO_SOT_SMD:SOT-23-5
- Y1: footprint (none) -> Crystal:Crystal_SMD_3225-4Pin_3.2x2.5mm_HandSoldering
Other:
- moved on the sheet: C1, C10, C11, C12, C13, C14, C15, C16, C17, C18, C19, C2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

Commit message: feat: create pcb
Changed lines of the file:
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@@
 	(text "POWER"
 		(exclude_from_sim no)
-		(at 574.294 173.99 0)
+		(at 592.074 173.736 0)
 		(effects
 			(font

Commit message: feat: component arrangement progress 1
Connections:
- net at D13.3 (DIN): no longer D12.1 (DOUT)
Changed lines of the file:
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@@
 	(wire
 		(pts
-			(xy 69.85 30.48) (xy 78.74 30.48)
+			(xy 69.85 30.48) (xy 60.96 30.48)
 		)
 		(stroke
